File: hardware/Power.kicad_sch (KiCad schematic)
At the start: 21 parts, among them J201 4090 USB-C, J202 9V battery, U201 LP2954AIT/NOPB

Commit message: Update design files to reflect new name
Other:
- company: (none) -> Finite Devices
- title: (none) -> Alethia

Commit message: Fix typo in branding files
Other:
- title: Alethia -> Aletheia
