File: hardware/Aletheia.kicad_pcb (KiCad board)
At the start: 12 copper layers, 94 x 127 mm, 85 parts, among them J101 Conn_01x04, J201 4090 USB-C, J202 9V battery, SW101 SW_DIP_x08, SW102 SW_DIP_x08, SW104 SW_DIP_x04, SW105 G19AP, SW301 Q/1/STOP, SW302 W/2/CH0, SW303 E/3/CH1, SW304 R/4/CH2, SW305 T/5/CH3, SW306 Y/6/_, SW307 U/7/-, SW308 I/8/+, SW309 O/9/=, SW310 P/0, SW311 A/!/`, SW312 S/"/CH4, SW313 D/$/CH5, SW314 F/%/CH6, SW315 G/^/CH7, SW316 H/&/{, SW317 J/*/}, SW318 K/(/[, SW319 L/)/], SW320 BKSP/DEL, SW321 SHIFT, SW322 Z/\/|, SW323 X/;/:, SW324 C/'/@, SW325 V/#/~, SW326 B/,/<, SW327 N/./>, SW328 M///?, SW329 SYM, SW330 SPC/ENT, U101 W65C02S6TPG-14, U102 AS6C1008-55PCN, U103 W65C22N6TPG-14, U104 74LS04, U105 74LS08, U106 74LS21, U201 LP2954AIT/NOPB, U301 MCP23S17_SP, U302 NHD-0420DZ-NSW-BBW, Y101 ECS-100AX-010

Commit message: Fix order of DIP switch lines in hardware
Connections:
- RN101 pad 2: /A7 -> /A0
- RN101 pad 3: /A6 -> /A1
- RN101 pad 4: /A5 -> /A2
- RN101 pad 5: /A4 -> /A3
- RN101 pad 6: /A3 -> /A4
- RN101 pad 7: /A2 -> /A5
- RN101 pad 8: /A1 -> /A6
- RN101 pad 9: /A0 -> /A7
- RN102 pad 2: /D7 -> /D0
- RN102 pad 3: /D6 -> /D1
- RN102 pad 4: /D5 -> /D2
- RN102 pad 5: /D4 -> /D3
- RN102 pad 6: /D3 -> /D4
- RN102 pad 7: /D2 -> /D5
- RN102 pad 8: /D1 -> /D6
- RN102 pad 9: /D0 -> /D7
- SW101 pad 10: /A6 -> /A1
- SW101 pad 11: /A5 -> /A2
- SW101 pad 12: /A4 -> /A3
- SW101 pad 13: /A3 -> /A4
- SW101 pad 14: /A2 -> /A5
- SW101 pad 15: /A1 -> /A6
- SW101 pad 16: /A0 -> /A7
- SW101 pad 9: /A7 -> /A0
- SW102 pad 10: /D6 -> /D1
- SW102 pad 11: /D5 -> /D2
- SW102 pad 12: /D4 -> /D3
- SW102 pad 13: /D3 -> /D4
- SW102 pad 14: /D2 -> /D5
- SW102 pad 15: /D1 -> /D6
- SW102 pad 16: /D0 -> /D7
- SW102 pad 9: /D7 -> /D0
Routing:
- net /D0: track 111.3 -> 173.2 mm
- net /D1: track 111.0 -> 167.5 mm
- net /D3: track 134.1 -> 184.6 mm
- net /D2: track 111.7 -> 162.0 mm
- net /D4: track 134.1 -> 179.3 mm
- net /D5: track 133.8 -> 173.9 mm
- net /D6: track 133.8 -> 167.8 mm
- net /A4: track 31.5 -> 62.6 mm
- net /D7: track 134.7 -> 162.2 mm
- net /A3: track 78.5 -> 104.2 mm
- net /A2: track 78.5 -> 98.8 mm
- net /A7: track 31.5 -> 47.9 mm
- net /A1: track 78.5 -> 93.5 mm
- net /A6: track 31.5 -> 42.5 mm
- net /A0: track 78.5 -> 89.3 mm
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